Commit message: Support workspace-provided Gazebo controllers and mode-matched command interfaces
Three fixes needed to drive the LBR from an external workspace:

- Plumb a `gazebo_controllers_path` xacro arg from each robot's top-level
  xacro through `*_description.xacro` into `lbr_gazebo.xacro`, so the
  gz_ros2_control plugin can load a workspace-specific controllers.yaml
  instead of the hardcoded one in lbr_description.
- Emit the command interface that matches `client_command_mode` in gazebo
  mode. Previously gazebo always got position only, so torque-mode
  simulation had no effort interface to claim.
- Rework `verify_joint_command_interfaces_()` to check for exactly one
  position and one effort interface by name rather than asserting on the
  raw count first, which produced a misleading error message.

Also refreshes the mock.rviz bringup config.

Co-Authored-By: Claude Opus 5 <noreply@anthropic.com>

File: lbr_description/gazebo/lbr_gazebo.xacro (robot description, xacro)
@@ -1,10 +1,11 @@
 <?xml version="1.0"?>
 <robot xmlns:xacro="http://www.ros.org/wiki/xacro">
-    <xacro:macro name="lbr_gazebo" params="robot_name:=^|lbr">
+    <xacro:macro name="lbr_gazebo"
+        params="robot_name:=^|lbr gazebo_controllers_path:=^|'$(find lbr_description)/ros2_control/lbr_controllers.yaml'">
         <!-- ros_control-plugin -->
         <gazebo>
             <plugin name="gz_ros2_control::GazeboSimROS2ControlPlugin"
                 filename="gz_ros2_control-system">
-                <parameters>$(find lbr_description)/ros2_control/lbr_controllers.yaml</parameters>
+                <parameters>${gazebo_controllers_path}</parameters>
                 <ros>
                     <namespace>/${robot_name}</namespace>

File: lbr_description/ros2_control/lbr_system_interface.xacro (robot description, xacro)
@@ -93,16 +93,18 @@
                 params="name min_position max_position max_velocity max_torque mode initial_position">
                 <joint name="${name}">
-                    <command_interface name="position">
+                    <xacro:if
+                        value="${mode != 'gazebo' or system_config['hardware']['client_command_mode'] == 'position'}">
+                        <command_interface name="position">
                         <param name="min">${min_position}</param>
                         <param name="max">${max_position}</param>
-                    </command_interface>
-                    <!-- only single command interface, refer
-                    https://github.com/ros-controls/gz_ros2_control/issues/182 -->
-                    <xacro:unless value="${mode == 'gazebo'}">
+                        </command_interface>
+                    </xacro:if>
+                    <xacro:if
+                        value="${mode != 'gazebo' or system_config['hardware']['client_command_mode'] == 'torque'}">
                         <command_interface name="effort">
                             <param name="min">-${max_torque}</param>
                             <param name="max"> ${max_torque}</param>
                         </command_interface>
-                    </xacro:unless>
+                    </xacro:if>
                     <state_interface name="position">
                       <param name="initial_value">${initial_position}</param>

File: lbr_description/urdf/iiwa14/iiwa14.xacro (robot description, xacro)
@@ -12,4 +12,7 @@
         name="initial_joint_positions_path"
         default="$(find lbr_description)/ros2_control/initial_joint_positions.yaml" />
+    <xacro:arg
+        name="gazebo_controllers_path"
+        default="$(find lbr_description)/ros2_control/lbr_controllers.yaml" />
     <!-- KDL requires a link without inertia / Gazebo requires a connection to world link or robot
     will tipple https://github.com/lbr-stack/lbr_fri_ros2_stack/issues/230 -->
@@ -26,4 +29,5 @@
         mode="$(arg mode)"
         system_config_path="$(arg system_config_path)"
-        initial_joint_positions_path="$(arg initial_joint_positions_path)" />
+        initial_joint_positions_path="$(arg initial_joint_positions_path)"
+        gazebo_controllers_path="$(arg gazebo_controllers_path)" />
 </robot>

File: lbr_description/urdf/iiwa14/iiwa14_description.xacro (robot description, xacro)
@@ -3,5 +3,5 @@
     <!-- robot as extracted via https://github.com/syuntoku14/fusion2urdf -->
     <xacro:macro name="iiwa14"
-        params="robot_name:=^|lbr mode:=^|mock system_config_path:=^|'$(find lbr_description)/ros2_control/lbr_system_config.yaml' initial_joint_positions_path:=^|'$(find lbr_description)/ros2_control/initial_joint_positions.yaml'">
+        params="robot_name:=^|lbr mode:=^|mock system_config_path:=^|'$(find lbr_description)/ros2_control/lbr_system_config.yaml' initial_joint_positions_path:=^|'$(find lbr_description)/ros2_control/initial_joint_positions.yaml' gazebo_controllers_path:=^|'$(find lbr_description)/ros2_control/lbr_controllers.yaml'">
         <!-- includes -->
         <xacro:include filename="$(find lbr_description)/gazebo/lbr_gazebo.xacro" />
@@ -16,5 +16,7 @@
         <xacro:property name="joint_friction" value="0.1" />
         <!-- macros for gazebo / mock / hardware -->
-        <xacro:lbr_gazebo robot_name="${robot_name}" />
+        <xacro:lbr_gazebo
+            robot_name="${robot_name}"
+            gazebo_controllers_path="${gazebo_controllers_path}" />
         <xacro:lbr_system_interface
             robot_name="${robot_name}"

File: lbr_description/urdf/iiwa7/iiwa7.xacro (robot description, xacro)
@@ -12,4 +12,7 @@
         name="initial_joint_positions_path"
         default="$(find lbr_description)/ros2_control/initial_joint_positions.yaml" />
+    <xacro:arg
+        name="gazebo_controllers_path"
+        default="$(find lbr_description)/ros2_control/lbr_controllers.yaml" />
     <!-- KDL requires a link without inertia / Gazebo requires a connection to world link or robot
     will tipple https://github.com/lbr-stack/lbr_fri_ros2_stack/issues/230 -->
@@ -26,4 +29,5 @@
         mode="$(arg mode)"
         system_config_path="$(arg system_config_path)"
-        initial_joint_positions_path="$(arg initial_joint_positions_path)" />
+        initial_joint_positions_path="$(arg initial_joint_positions_path)"
+        gazebo_controllers_path="$(arg gazebo_controllers_path)" />
 </robot>

File: lbr_description/urdf/iiwa7/iiwa7_description.xacro (robot description, xacro)
@@ -3,5 +3,5 @@
     <!-- robot as extracted via https://github.com/syuntoku14/fusion2urdf -->
     <xacro:macro name="iiwa7"
-        params="robot_name:=^|lbr mode:=^|mock system_config_path:=^|'$(find lbr_description)/ros2_control/lbr_system_config.yaml' initial_joint_positions_path:=^|'$(find lbr_description)/ros2_control/initial_joint_positions.yaml'">
+        params="robot_name:=^|lbr mode:=^|mock system_config_path:=^|'$(find lbr_description)/ros2_control/lbr_system_config.yaml' initial_joint_positions_path:=^|'$(find lbr_description)/ros2_control/initial_joint_positions.yaml' gazebo_controllers_path:=^|'$(find lbr_description)/ros2_control/lbr_controllers.yaml'">
         <!-- includes -->
         <xacro:include filename="$(find lbr_description)/gazebo/lbr_gazebo.xacro" />
@@ -16,5 +16,7 @@
         <xacro:property name="joint_friction" value="0.1" />
         <!-- macros for gazebo / mock / hardware -->
-        <xacro:lbr_gazebo robot_name="${robot_name}" />
+        <xacro:lbr_gazebo
+            robot_name="${robot_name}"
+            gazebo_controllers_path="${gazebo_controllers_path}" />
         <xacro:lbr_system_interface
             robot_name="${robot_name}"

File: lbr_description/urdf/med14/med14.xacro (robot description, xacro)
@@ -12,4 +12,7 @@
         name="initial_joint_positions_path"
         default="$(find lbr_description)/ros2_control/initial_joint_positions.yaml" />
+    <xacro:arg
+        name="gazebo_controllers_path"
+        default="$(find lbr_description)/ros2_control/lbr_controllers.yaml" />
     <!-- KDL requires a link without inertia / Gazebo requires a connection to world link or robot
     will tipple https://github.com/lbr-stack/lbr_fri_ros2_stack/issues/230 -->
@@ -26,4 +29,5 @@
         mode="$(arg mode)"
         system_config_path="$(arg system_config_path)"
-        initial_joint_positions_path="$(arg initial_joint_positions_path)" />
+        initial_joint_positions_path="$(arg initial_joint_positions_path)"
+        gazebo_controllers_path="$(arg gazebo_controllers_path)" />
 </robot>

File: lbr_description/urdf/med14/med14_description.xacro (robot description, xacro)
@@ -3,5 +3,5 @@
     <!-- robot as extracted via https://github.com/syuntoku14/fusion2urdf -->
     <xacro:macro name="med14"
-        params="robot_name:=^|lbr mode:=^|mock system_config_path:=^|'$(find lbr_description)/ros2_control/lbr_system_config.yaml' initial_joint_positions_path:=^|'$(find lbr_description)/ros2_control/initial_joint_positions.yaml'">
+        params="robot_name:=^|lbr mode:=^|mock system_config_path:=^|'$(find lbr_description)/ros2_control/lbr_system_config.yaml' initial_joint_positions_path:=^|'$(find lbr_description)/ros2_control/initial_joint_positions.yaml' gazebo_controllers_path:=^|'$(find lbr_description)/ros2_control/lbr_controllers.yaml'">
         <!-- includes -->
         <xacro:include filename="$(find lbr_description)/gazebo/lbr_gazebo.xacro" />
@@ -16,5 +16,7 @@
         <xacro:property name="joint_friction" value="0.1" />
         <!-- macros for gazebo / mock / hardware -->
-        <xacro:lbr_gazebo robot_name="${robot_name}" />
+        <xacro:lbr_gazebo
+            robot_name="${robot_name}"
+            gazebo_controllers_path="${gazebo_controllers_path}" />
         <xacro:lbr_system_interface
             robot_name="${robot_name}"

File: lbr_description/urdf/med7/med7.xacro (robot description, xacro)
@@ -12,4 +12,7 @@
         name="initial_joint_positions_path"
         default="$(find lbr_description)/ros2_control/initial_joint_positions.yaml" />
+    <xacro:arg
+        name="gazebo_controllers_path"
+        default="$(find lbr_description)/ros2_control/lbr_controllers.yaml" />
     <!-- KDL requires a link without inertia / Gazebo requires a connection to world link or robot
     will tipple https://github.com/lbr-stack/lbr_fri_ros2_stack/issues/230 -->
@@ -26,4 +29,5 @@
         mode="$(arg mode)"
         system_config_path="$(arg system_config_path)"
-        initial_joint_positions_path="$(arg initial_joint_positions_path)" />
+        initial_joint_positions_path="$(arg initial_joint_positions_path)"
+        gazebo_controllers_path="$(arg gazebo_controllers_path)" />
 </robot>

File: lbr_description/urdf/med7/med7_description.xacro (robot description, xacro)
@@ -3,5 +3,5 @@
     <!-- robot as extracted via https://github.com/syuntoku14/fusion2urdf -->
     <xacro:macro name="med7"
-        params="robot_name:=^|lbr mode:=^|mock system_config_path:=^|'$(find lbr_description)/ros2_control/lbr_system_config.yaml' initial_joint_positions_path:=^|'$(find lbr_description)/ros2_control/initial_joint_positions.yaml'">
+        params="robot_name:=^|lbr mode:=^|mock system_config_path:=^|'$(find lbr_description)/ros2_control/lbr_system_config.yaml' initial_joint_positions_path:=^|'$(find lbr_description)/ros2_control/initial_joint_positions.yaml' gazebo_controllers_path:=^|'$(find lbr_description)/ros2_control/lbr_controllers.yaml'">
         <!-- includes -->
         <xacro:include filename="$(find lbr_description)/gazebo/lbr_gazebo.xacro" />
@@ -16,5 +16,7 @@
         <xacro:property name="joint_friction" value="0.1" />
         <!-- macros for gazebo / mock / hardware -->
-        <xacro:lbr_gazebo robot_name="${robot_name}" />
+        <xacro:lbr_gazebo
+            robot_name="${robot_name}"
+            gazebo_controllers_path="${gazebo_controllers_path}" />
         <xacro:lbr_system_interface
             robot_name="${robot_name}"
